File: board/board.kicad_pcb (KiCad board)
At the start: 2 copper layers, 21 x 13 mm, 1 part

Commit message: initial
Parts:
- removed LOGO1: Logo_Open_Hardware_Small, Symbol:OSHW-Symbol_6.7x6mm_SilkScreen
- added C1: 100nF, Capacitor_SMD:C_0603_1608Metric, F.Cu at (33.4, 169.2)
- added C2: 220nF, Capacitor_SMD:C_0603_1608Metric, F.Cu at (33.4, 167.4)
- added C3: 100nF, Capacitor_SMD:C_0603_1608Metric, F.Cu at (44.4, 168.9)
- added C4: 100nF, Capacitor_SMD:C_0603_1608Metric, F.Cu at (32.1, 162.0)
- added J1: 002_SPI, on_edge:on_edge_2x05_device, F.Cu at (30.0, 153.5)
- added J2: 007_ADC, on_edge:on_edge_2x05_host, F.Cu at (51.0, 153.5)
- added J3: 007_ADC, on_edge:on_edge_2x05_host, F.Cu at (51.0, 170.0)
- added U1: ADS131M04, Package_SO:TSSOP-20_4.4x6.5mm_P0.65mm, F.Cu at (39.5, 165.3)
- added X1: 8MhZ, Oscillator:Oscillator_SMD_EuroQuartz_XO32-4Pin_3.2x2.5mm, F.Cu at (32.1, 164.7)
- added l1: Logo_Open_Hardware_Larg, Symbol:OSHW-Logo2_7.3x6mm_SilkScreen, F.Cu at (34.3, 173.0)
Routing:
- net GND: track 0.00 -> 62.6 mm, vias 0 -> 30
- net /3.3V: track 0.00 -> 58.2 mm, vias 0 -> 5
- net /5V: track 0.00 -> 35.7 mm
- net /ADC/MOSI: track 0.00 -> 19.1 mm
- net /ADC/AD4-: track 0.00 -> 19.1 mm, vias 0 -> 1
- net /ADC/CS: track 0.00 -> 17.4 mm, vias 0 -> 1
- net /ADC/MISO: track 0.00 -> 16.5 mm
- net /ADC/SCLK: track 0.00 -> 16.3 mm
- net /ADC/AD3+: track 0.00 -> 15.7 mm
- net /ADC//DRDY: track 0.00 -> 15.5 mm
- net /ADC/AD2+: track 0.00 -> 15.5 mm, vias 0 -> 2
- net /ADC/AD3-: track 0.00 -> 15.0 mm
- net /ADC//RESET: track 0.00 -> 13.6 mm, vias 0 -> 1
- net /ADC/AD4+: track 0.00 -> 12.0 mm
- net /ADC/AD1-: track 0.00 -> 10.4 mm, vias 0 -> 2
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- added copper zone on B.Cu, net GND
- added copper zone on F.Cu, net GND
Other:
- board size 21 x 13 mm -> 21 x 28.8 mm
- rule pad_to_mask_clearance: 0 -> 0.04
- board text added: "osf.002"
- board text added: "osf.007"
- board text added: "osf.b084.v1.0"
